File: Kicad/Carte_Ucontroleur/Merx_Carte_Ucontroleur.kicad_pcb (KiCad board)
At the start: 2 copper layers, 75.1 x 65 mm, 22 parts, among them IC1 TCA9545APWR, J1 Autocom3, J10 Mouting_Screw_3mm, J11 Grove, J12 Autocom2, J13 Autocom2, J3 Autocom4, J4 Grove, J5 Grove, J6 Grove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

Commit message: Nouveau kIcad corrigé
Parts:
- removed J1: Autocom3, FootprintGamelGe2_v6:Autocom3
- added J14: Autocom2, FootprintGamelGe2_v6:Autocom2, F.Cu at (119.5, 91.0)
- added Q1: NX3008NBK, NX3008NBK:SOT23-3, F.Cu at (114.7, 91.5)
- added Q2: PMEG2020AEA, PMEG2020AEA:DIO_BZX384-C30_115, F.Cu at (109.9, 92.1)
- added R2: 10k, Resistor_SMD:R_1206_3216Metric, F.Cu at (109.8, 88.1)
- added R3: 100 ou 330, Resistor_SMD:R_1206_3216Metric, F.Cu at (115.0, 88.2)
- turned J11 to 90 degrees
- turned J4 to 0 degrees
- turned J5 to 0 degrees
- turned J6 to -90 degrees
- turned J7 to -90 degrees
Connections:
- U5 pad 3: /encodeur_2 + -> /encodeur_2 -
- U5 pad 4: /encodeur_2 - -> /encodeur_2 +
- U5 pad 5: /encodeur_1 + -> /encodeur_1 -
- U5 pad 6: /encodeur_1 - -> /encodeur_1 +
- U5 pad 7: /servo -> /on/off servo
Routing:
- net GND: track 411.4 -> 485.6 mm, vias 6 -> 7
- net /Rx: track 123.9 -> 104.9 mm
- net /on/off servo: track 0.00 -> 17.6 mm, vias 0 -> 1
- net /Tx: track 118.8 -> 101.3 mm
- net /scl1: track 31.1 -> 38.9 mm
- net +5V: track 151.9 -> 156.8 mm, vias 0 -> 1
- net /scl0: track 32.4 -> 28.0 mm
- net /servo: track 12.9 -> 17.0 mm, vias 0 -> 1
- net /encodeur_1 +: track 46.8 -> 42.9 mm
- net /encodeur_1 -: track 42.9 -> 46.8 mm
- net /encodeur_2 -: track 17.5 -> 14.0 mm
- net /encodeur_2 +: track 14.0 -> 17.5 mm
- net +3.3V_ESP: track 132.5 -> 129.1 mm, vias 1 -> 2
- net Net-(Q1-Pad1): track 0.00 -> 3.06 mm
- net /sda1: track 33.4 -> 36.0 mm
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