File: Kicad/Carte_Ucontroleur/Merx_Carte_Ucontroleur.kicad_sch (KiCad schematic)
At the start: 22 parts, among them IC1 TCA9545APWR, J1 Autocom3, J10 Mouting_Screw_3mm, J11 Grove, J12 Autocom2, J13 Autocom2, J3 Autocom4, J4 Grove, J5 Grove, J6 Grove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

Commit message: Nouveau kIcad corrigé
Parts:
- removed J1: Autocom3, FootprintGamelGe2_v6:Autocom3, symbol SymbGamelGe2_v6:Autocom3
- added J14: Autocom2, FootprintGamelGe2_v6:Autocom2, symbol SymbGamelGe2_v6:Autocom2
- added Q1: NX3008NBK, NX3008NBK:SOT23-3, symbol NX3008NBK:NX3008NBK
- added Q2: PMEG2020AEA, PMEG2020AEA:DIO_BZX384-C30_115, symbol PMEG2020AEA:PMEG2020AEA
- added R2: 10k, Resistor_SMD:R_1206_3216Metric, symbol SymbGamelGe2_v6:R
- added R3: 100 ou 330, Resistor_SMD:R_1206_3216Metric, symbol SymbGamelGe2_v6:R
Connections:
- net +5V: now also J14.1 (Pin_1), Q2.K
- net GND: now also Q1.2, R2.2
- net encodeur_1 +: now also U5.6 (IO35); no longer U5.5 (IO34)
- net encodeur_1 -: now also U5.5 (IO34); no longer U5.6 (IO35)
- net encodeur_2 +: now also U5.4 (SENSOR_VN); no longer U5.3 (SENSOR_VP)
- net encodeur_2 -: now also U5.3 (SENSOR_VP); no longer U5.4 (SENSOR_VN)
- net servo: now also J14.2 (Pin_2), Q1.3, Q2.A; no longer U5.7 (IO32)
- new net: Q1.1, R3.2
- new net on/off servo: R2.1, R3.1, U5.7 (IO32)
Other:
- note added: "Tourni !"
- note removed: "Servo Fin"
- moved on the sheet: J12, J6
